File: lichen-badge.kicad_pcb (KiCad board)
At the start: 2 copper layers, 96.3 x 113 mm, 10 parts, among them J1 Micro_SD_Card_Det, J2 USB_A, J3 USB_B_Micro, U1 OSD335x-CSIP, U2 MMA8452QR1

Commit message: Update schematic for Octavo review
Signed-off-by: Michael Welling <mwelling@ieee.org>
Parts:
- J3: footprint lichen-badge:10118192-0001LF(MICRO-USB-B-AMPHENOL-FCI) -> Connector_USB:USB_Micro-B_Molex-105017-0001
- moved J1 79.1 mm to (153.9, 153.3), turned to 0 degrees
- moved J3 72.9 mm to (114.6, 180.2), turned to 0 degrees
- moved J2 42.6 mm to (93.7, 173.6), turned to 0 degrees
- moved U2 32.0 mm to (119.0, 133.6)
Connections:
- net Net-(U1-PadB17) renamed WARMRSTN
- net Net-(U1-PadC17) renamed PWRONRSTN_OD
- net Net-(U1-PadH1) renamed USB1_VBUS
- net Net-(U1-PadH3) renamed USB1_DRVVBUS
- net Net-(U1-PadV4) renamed MMC0_CD
- net Net-(U1-PadW6) renamed UART0_TXD
- net Net-(U1-PadY6) renamed UART0_RXD
- J1 pad 1: Net-(J1-Pad1) -> MMC0_DAT2
- J1 pad 2: Net-(J1-Pad2) -> MMC0_DAT3
- J1 pad 3: Net-(J1-Pad3) -> MMC0_CMD
- J1 pad 4: Net-(J1-Pad4) -> SYS_VDD1_3P3V
- J1 pad 5: Net-(J1-Pad5) -> MMC0_CLK
- J1 pad 6: Net-(J1-Pad6) -> GND
- J1 pad 7: Net-(J1-Pad7) -> MMC0_DAT0
- J1 pad 8: Net-(J1-Pad8) -> MMC0_DAT1
- J1 pad 9: Net-(J1-Pad9) -> GND
- J2 pad 2: Net-(J2-Pad2) -> USB1_DM
- J2 pad 3: Net-(J2-Pad3) -> USB1_DP
- J2 pad 4: Net-(J2-Pad4) -> GND
- J2 pad 5: Net-(J2-Pad5) -> GNDPWR
- U1 pad B18: Net-(U1-PadB18) -> USB0_VBUS
- U1 pad B19: Net-(U1-PadB19) -> USB0_VBUS
- U1 pad B20: Net-(U1-PadB20) -> USB0_VBUS
- U1 pad C18: Net-(U1-PadC18) -> VIN_AC
- U1 pad C19: Net-(U1-PadC19) -> VIN_AC
- U1 pad C20: Net-(U1-PadC20) -> VIN_AC
- U1 pad D12: Net-(U1-PadD12) -> Net-(U1-PadD11)
- U1 pad D14: Net-(U1-PadD14) -> Net-(U1-PadD13)
- U1 pad D18: Net-(U1-PadD18) -> VBAT
- U1 pad D19: Net-(U1-PadD19) -> VBAT
- U1 pad D20: Net-(U1-PadD20) -> VBAT
- U1 pad D9: Net-(U1-PadD9) -> Net-(U1-PadD10)
- U1 pad E19: Net-(U1-PadE19) -> VBAT
- U1 pad F12: Net-(U1-PadF12) -> SYS_VDD2_3P3V
- U1 pad F13: Net-(U1-PadF13) -> SYS_VDD2_3P3V
- U1 pad F14: Net-(U1-PadF14) -> SYS_VOUT
- U1 pad F15: Net-(U1-PadF15) -> SYS_VOUT
- U1 pad F8: Net-(U1-PadF8) -> SYS_VDD1_3P3V
- U1 pad F9: Net-(U1-PadF9) -> SYS_VDD1_3P3V
- U1 pad G12: Net-(U1-PadG12) -> SYS_VDD2_3P3V
- U1 pad G13: Net-(U1-PadG13) -> SYS_VDD2_3P3V
- U1 pad G14: Net-(U1-PadG14) -> SYS_VOUT
- U1 pad G15: Net-(U1-PadG15) -> SYS_VOUT
- U1 pad G8: Net-(U1-PadG8) -> SYS_VDD1_3P3V
- U1 pad G9: Net-(U1-PadG9) -> SYS_VDD1_3P3V
- U1 pad H14: Net-(U1-PadH14) -> SYS_VDD1_3P3V
- U1 pad H15: Net-(U1-PadH15) -> SYS_VDD1_3P3V
- U1 pad H17: Net-(U1-PadH17) -> Net-(U1-PadG17)
- U1 pad H2: Net-(U1-PadH2) -> USB1_DM
- U1 pad H7: Net-(U1-PadH7) -> SYS_VDD1_3P3V
- U1 pad H8: Net-(U1-PadH8) -> SYS_VDD1_3P3V
- U1 pad J1: Net-(U1-PadJ1) -> GND
- U1 pad J14: Net-(U1-PadJ14) -> SYS_VDD1_3P3V
- U1 pad J15: Net-(U1-PadJ15) -> SYS_VDD1_3P3V
- U1 pad J2: Net-(U1-PadJ2) -> USB1_DP
- U1 pad J7: Net-(U1-PadJ7) -> SYS_VDD1_3P3V
- U1 pad J8: Net-(U1-PadJ8) -> SYS_VDD1_3P3V
- U1 pad K1: Net-(U1-PadK1) -> USB0_VBUS
- U1 pad K10: Net-(U1-PadK10) -> SYS_VDD3_3P3V
- U1 pad K11: Net-(U1-PadK11) -> SYS_VDD3_3P3V
- U1 pad K13: Net-(U1-PadK13) -> SYS_VDD_1P8V
- U1 pad K14: Net-(U1-PadK14) -> SYS_VDD_1P8V
- U1 pad K17: Net-(U1-PadK17) -> Net-(U1-PadJ17)
- U1 pad K2: Net-(U1-PadK2) -> USB0_DM
- U1 pad L1: Net-(U1-PadL1) -> USB0_ID
- U1 pad L10: Net-(U1-PadL10) -> SYS_VDD3_3P3V
- U1 pad L11: Net-(U1-PadL11) -> SYS_VDD3_3P3V
- U1 pad L12: Net-(U1-PadL12) -> SYS_VDD3_3P3V
- U1 pad L13: Net-(U1-PadL13) -> SYS_VDD_1P8V
- U1 pad L14: Net-(U1-PadL14) -> SYS_VDD_1P8V
- U1 pad L2: Net-(U1-PadL2) -> USB0_DP
- U1 pad L7: Net-(U1-PadL7) -> SYS_VDD3_3P3V
- U1 pad L8: Net-(U1-PadL8) -> SYS_VDD3_3P3V
- U1 pad L9: Net-(U1-PadL9) -> SYS_VDD3_3P3V
- U1 pad M10: Net-(U1-PadM10) -> SYS_VDD3_3P3V
- U1 pad M11: Net-(U1-PadM11) -> SYS_VDD3_3P3V
- U1 pad M12: Net-(U1-PadM12) -> SYS_VDD3_3P3V
- U1 pad M13: Net-(U1-PadM13) -> SYS_VDD_1P8V
- U1 pad M14: Net-(U1-PadM14) -> SYS_VDD_1P8V
- U1 pad M7: Net-(U1-PadM7) -> SYS_VDD3_3P3V
- U1 pad M8: Net-(U1-PadM8) -> SYS_VDD3_3P3V
- U1 pad M9: Net-(U1-PadM9) -> SYS_VDD3_3P3V
- U1 pad N10: Net-(U1-PadN10) -> SYS_VDD_1P8V
- U1 pad N11: Net-(U1-PadN11) -> SYS_VDD_1P8V
- U1 pad N12: Net-(U1-PadN12) -> SYS_VDD_1P8V
- U1 pad N13: Net-(U1-PadN13) -> SYS_VDD_1P8V
- U1 pad N14: Net-(U1-PadN14) -> SYS_VDD_1P8V
- U1 pad N7: Net-(U1-PadN7) -> SYS_VDD_1P8V
- U1 pad N8: Net-(U1-PadN8) -> SYS_VDD_1P8V
- U1 pad N9: Net-(U1-PadN9) -> SYS_VDD_1P8V
- U1 pad P10: Net-(U1-PadP10) -> SYS_VDD_1P8V
- U1 pad P11: Net-(U1-PadP11) -> SYS_VDD_1P8V
- U1 pad U15: Net-(U1-PadU15) -> GND
- U1 pad V2: Net-(U1-PadV2) -> MMC0_DAT2
- U1 pad V3: Net-(U1-PadV3) -> MMC0_DAT1
- U1 pad V7: Net-(U1-PadV7) -> Net-(U1-PadU7)
- U1 pad V8: Net-(U1-PadV8) -> Net-(U1-PadU8)
- U1 pad W2: Net-(U1-PadW2) -> MMC0_CMD
- U1 pad W3: Net-(U1-PadW3) -> MMC0_CLK
- U1 pad W7: Net-(U1-PadW7) -> I2C1_SCL
- U1 pad Y2: Net-(U1-PadY2) -> MMC0_DAT3
- U1 pad Y3: Net-(U1-PadY3) -> MMC0_DAT0
- U1 pad Y7: Net-(U1-PadY7) -> I2C1_SDA
- U2 pad 1: Net-(U2-Pad1) -> SYS_VDD1_3P3V
- U2 pad 10: Net-(U2-Pad10) -> GND
- U2 pad 12: Net-(U2-Pad12) -> GND
- U2 pad 14: Net-(U2-Pad14) -> SYS_VDD1_3P3V
- U2 pad 4: Net-(U2-Pad4) -> I2C1_SCL
- U2 pad 5: Net-(U2-Pad5) -> GND
- U2 pad 6: Net-(U2-Pad6) -> I2C1_SDA
- U2 pad 7: Net-(U2-Pad7) -> GND

Commit message: Design released to OSHPark
Hope it works. :)

Signed-off-by: Michael Welling <mwelling@ieee.org>
Parts:
- added C1: 22uF, Capacitor_SMD:C_0805_2012Metric, F.Cu at (70.2, 123.1)
- added C2: 22uF, Capacitor_SMD:C_0805_2012Metric, F.Cu at (71.7, 138.2)
- added C3: 22uF, Capacitor_SMD:C_0805_2012Metric, F.Cu at (71.7, 140.6)
- added C4: .1uF, Capacitor_SMD:C_0402_1005Metric, F.Cu at (119.5, 129.7)
- added C5: .1uF, Capacitor_SMD:C_0402_1005Metric, F.Cu at (115.0, 133.1)
- added C6: 10uF, Capacitor_SMD:C_0805_2012Metric, F.Cu at (114.8, 149.9)
- added C7: .1uF, Capacitor_SMD:C_0402_1005Metric, F.Cu at (114.8, 151.7)
- added C9: 47uF, Inductor_SMD:L_0805_2012Metric, F.Cu at (94.5, 119.8)
- added D1: LED_RABG, lichen-badge:LED_SunLED_PLCC4_3.2x2.8mm_Reverse_Mount, F.Cu at (95.1, 83.9)
- added D2: LED_RABG, lichen-badge:LED_SunLED_PLCC4_3.2x2.8mm_Reverse_Mount, F.Cu at (109.5, 83.3)
- added FB1: Ferrite_Bead_Small, Inductor_SMD:L_0603_1608Metric, F.Cu at (101.4, 160.9)
- added FB2: Ferrite_Bead_Small, Inductor_SMD:L_0603_1608Metric, F.Cu at (87.7, 160.9)
- added FB3: Ferrite_Bead_Small, Inductor_SMD:L_0603_1608Metric, F.Cu at (106.3, 160.9)
- added FB4: Ferrite_Bead_Small, Inductor_SMD:L_0603_1608Metric, F.Cu at (92.7, 160.9)
- added H1: MountingHole, MountingHole:MountingHole_6.5mm, F.Cu at (100.1, 65.7)
- added IC1: TPD4S012DRYR, lichen-badge:SON-6(TI)-DRY, F.Cu at (90.1, 160.8)
- added IC2: TPD4S012DRYR, lichen-badge:SON-6(TI)-DRY, F.Cu at (103.8, 160.7)
- added J4: TEST_1P, TestPoint:TestPoint_Pad_D1.0mm, F.Cu at (103.4, 150.7)
- added J5: JST, Connector_JST:JST_PH_S2B-PH-SM4-TB_1x02-1MP_P2.00mm_Horizontal, F.Cu at (75.7, 117.0)
- added J6: Conn_01x04, Connector_Molex:Molex_PicoBlade_53261-0471_1x04-1MP_P1.25mm_Horizontal, F.Cu at (128.9, 129.4)
- added J7: TEST_1P, TestPoint:TestPoint_Pad_D1.0mm, F.Cu at (106.0, 150.7)
- added L1: 2.2uH, Inductor_SMD:L_Taiyo-Yuden_MD-4040, F.Cu at (70.6, 126.6)
- added Q1: MMBT3904, Package_TO_SOT_SMD:SOT-23, F.Cu at (123.0, 140.1)
- added Q2: MMBT3904, Package_TO_SOT_SMD:SOT-23, F.Cu at (85.3, 92.8)
- added Q3: MMBT3904, Package_TO_SOT_SMD:SOT-23, F.Cu at (85.3, 85.6)
- added Q4: MMBT3904, Package_TO_SOT_SMD:SOT-23, F.Cu at (85.3, 77.4)
- added R1: 10K, Resistor_SMD:R_0402_1005Metric, F.Cu at (92.9, 120.2)
- added R10: 4.7K, Resistor_SMD:R_0402_1005Metric, F.Cu at (114.8, 146.9)
- added R11: 4.7K, Resistor_SMD:R_0402_1005Metric, F.Cu at (111.0, 150.7)
- added R12: 4.7K, Resistor_SMD:R_0402_1005Metric, F.Cu at (114.8, 143.8)
- added R13: 4.7K, Resistor_SMD:R_0402_1005Metric, F.Cu at (109.7, 150.7)
- added R14: 4.7K, Resistor_SMD:R_0402_1005Metric, F.Cu at (108.5, 150.7)
- added R15: 470, Resistor_SMD:R_0402_1005Metric, F.Cu at (126.2, 141.0)
- added R16: 22, Resistor_SMD:R_0402_1005Metric, F.Cu at (119.8, 142.1)
- added R17: 4.7K, Resistor_SMD:R_0402_1005Metric, F.Cu at (85.9, 95.9)
- added R18: 4.7K, Resistor_SMD:R_0402_1005Metric, F.Cu at (85.9, 88.4)
- added R19: 4.7K, Resistor_SMD:R_0402_1005Metric, F.Cu at (85.9, 80.5)
- added R2: 750K, Resistor_SMD:R_0402_1005Metric, F.Cu at (70.5, 129.6)
- added R20: 100K, Resistor_SMD:R_0402_1005Metric, F.Cu at (85.9, 97.3)
- added R21: 100K, Resistor_SMD:R_0402_1005Metric, F.Cu at (85.9, 89.7)
- added R22: 100K, Resistor_SMD:R_0402_1005Metric, F.Cu at (85.9, 82.0)
- added R3: 750K, Resistor_SMD:R_0402_1005Metric, F.Cu at (68.4, 138.0)
- added R4: 100K, Resistor_SMD:R_0402_1005Metric, F.Cu at (67.2, 138.0)
- added R5: 4.7K, Resistor_SMD:R_0402_1005Metric, F.Cu at (115.6, 137.2)
- added R6: 4.7K, Resistor_SMD:R_0402_1005Metric, F.Cu at (119.0, 137.2)
- added R7: 100, Resistor_SMD:R_0402_1005Metric, F.Cu at (106.0, 111.0)
- added R8: 4.7K, Resistor_SMD:R_0402_1005Metric, F.Cu at (114.8, 142.3)
- added R9: 4.7K, Resistor_SMD:R_0402_1005Metric, F.Cu at (114.8, 145.3)
- added RN5: 470, Resistor_SMD:R_Array_Convex_4x0402, F.Cu at (95.2, 77.0)
- added RN6: 470, Resistor_SMD:R_Array_Convex_4x0402, F.Cu at (109.4, 77.0)
- added SW1: POWER, Button_Switch_SMD:SW_SPST_EVQP2, F.Cu at (87.1, 104.1)
- added SW2: RESET, Button_Switch_SMD:SW_SPST_EVQP2, F.Cu at (97.3, 104.1)
- added SW3: BOOT0, Button_Switch_SMD:SW_SPST_EVQP2, F.Cu at (108.0, 104.1)
- added U4: PAM2401SCADJ, Package_SO:MSOP-8_3x3mm_P0.65mm, F.Cu at (70.5, 133.8)
- added U5: TPS2051C, lichen-badge:SOT-23-5, F.Cu at (86.3, 157.1)
- added X1: SPI-LCD-(1.8IN), lichen-badge:LCD-(1.8IN), B.Cu at (97.7, 140.5)
- J1: footprint lichen-badge:MICROSD -> Connector_Card:microSD_HC_Hirose_DM3AT-SF-PEJM5
- J2: value USB_A -> USB_B_Micro; footprint Connectors:USB_A -> Connector_USB:USB_Micro-B_Molex_47346-0001
- J3: footprint Connector_USB:USB_Micro-B_Molex-105017-0001 -> Connector_USB:USB_Micro-B_Molex_47346-0001
- RN1, RN2, RN3, RN4: footprint Resistors_SMD:R_Array_Convex_4x0402 -> Resistor_SMD:R_Array_Convex_4x0402
- moved J1 32.9 mm to (122.4, 163.0), turned to 20 degrees
- moved J3 18.5 mm to (103.9, 165.2)
- moved J2 9.13 mm to (90.2, 165.2)
- moved U1 0.07 mm to (99.6, 135.6)
Connections:
- net USB0_DM renamed USB0_D-
- net USB0_DP renamed USB0_D+
- net USB1_DM renamed USB1_D-
- net USB1_DP renamed USB1_D+
- J2 pad 4: GND -> USB1_ID
- J2 pad 5: GNDPWR -> GND
- U1 pad A14: Net-(U1-PadA14) -> LCD_RS
- U1 pad A16: Net-(U1-PadA16) -> LCD_RESET
- U1 pad B17: WARMRSTN -> Net-(SW2-Pad2)
- U1 pad C13: Net-(U1-PadC13) -> PWM_BLUE
- U1 pad C17: PWRONRSTN_OD -> Net-(SW2-Pad2)
- U1 pad J1: GND -> USB1_ID
- U1 pad U20: Net-(U1-PadU20) -> LCD_PWM
- U1 pad V16: Net-(U1-PadV16) -> PWM_RED
- U1 pad W4: Net-(U1-PadW4) -> SPI0_MOSI
- U1 pad Y12: Net-(U1-PadY12) -> Net-(U1-PadW12)
- U1 pad Y16: Net-(U1-PadY16) -> PWM_GREEN
- U1 pad Y4: Net-(U1-PadY4) -> SPI0_nCS0
- U1 pad Y5: Net-(U1-PadY5) -> SPI0_SCLK
- U1 pad Y9: Net-(U1-PadY9) -> Net-(U1-PadW9)
Routing:
- net PWM_GREEN: track 0.00 -> 70.4 mm, vias 0 -> 2
- net VIN_AC: track 0.00 -> 66.1 mm, vias 0 -> 2
- net GND: track 0.00 -> 62.1 mm, vias 0 -> 142
- net PWM_BLUE: track 0.00 -> 61.4 mm, vias 0 -> 2
- net PWM_RED: track 0.00 -> 59.6 mm, vias 0 -> 2
- net VBAT: track 0.00 -> 48.2 mm
- net Net-(Q2-Pad3): track 0.00 -> 44.0 mm, vias 0 -> 3
- net VBOOST: track 0.00 -> 38.2 mm
- net LCD_RESET: track 0.00 -> 37.7 mm, vias 0 -> 1
- net Net-(Q3-Pad3): track 0.00 -> 37.6 mm, vias 0 -> 3
- net LCD_PWM: track 0.00 -> 36.7 mm, vias 0 -> 2
- net Net-(SW2-Pad2): track 0.00 -> 36.4 mm, vias 0 -> 2
- net SYS_VDD1_3P3V: track 0.00 -> 32.7 mm, vias 0 -> 20
- net LCD_RS: track 0.00 -> 32.2 mm, vias 0 -> 1
- net SYS_VOUT: track 0.00 -> 31.6 mm, vias 0 -> 3
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- added copper zone on F.Cu, net GND
- added copper zone on In2.Cu, net GND
- added copper zone on F.Cu, net GNDPWR
- added copper zone on In2.Cu, net GNDPWR
- added copper zone on B.Cu, net SYS_VDD1_3P3V
- added copper zone on F.Cu, net SYS_VDD1_3P3V
- added copper zone on In1.Cu, net SYS_VDD1_3P3V
- added copper zone on F.Cu, net SYS_VOUT
- added copper zone on In1.Cu, net SYS_VOUT
- added copper zone on In1.Cu, net USB0_VBUS
- added copper zone on F.Cu, net VIN_AC
Other:
- board size 96.3 x 113 mm -> 96.3 x 113.2 mm
- copper layers 2 -> 4
- net class Default: clearance 0.2 -> 0.1524; trace_width 0.25 -> 0.1524; via_dia 0.8 -> 0.508; via_drill 0.4 -> 0.254
- rule pad_to_mask_clearance: 0.2 -> 0.0254
- rule trace_clearance: 0.2 -> 0.1524
- rule trace_min: 0.2 -> 0.1524
- rule via_min_drill: 0.3 -> 0.254
- rule via_min_size: 0.4 -> 0.508
- board text added: "EEP"

Commit message: Add BOM for the design
Signed-off-by: Michael Welling <mwelling@ieee.org>
Parts:
- C9: footprint Inductor_SMD:L_0805_2012Metric -> Capacitor_SMD:C_0805_2012Metric
Changed lines of the file:
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@@
     (add_net VIN_AC)
+  )
+  (module Capacitor_SMD:C_0805_2012Metric (layer F.Cu)
+    (at 94.488 119.8118 90)
+    (descr "Capacitor SMD 0805 (2012 Metric), square (rectangular) end terminal, IPC_7351 nominal, (Body size source: https://docs.google.com/spreadsheets/d/1BsfQQcO9C6DZCsRaXUlFlo91Tg2WpOkGARC1WS5S8t0/edit?usp=sharing), generated with kicad-footprint-generator")
+    (tags capacitor)
+    (attr smd)
+    (fp_text reference C9 (at 2.794 0.0508 90) (layer F.SilkS)
+      (effects (font (size 1 1) (thickness 0.15)))
+    )
+    (fp_text value 47uF (at 0 1.65 90) (layer F.Fab)
+      (effects (font (size 1 1) (thickness 0.15)))
+    )
+    (fp_text user %R (at 0 0 90) (layer F.Fab)
+      (effects (font (size 0.5 0.5) (thickness 0.08)))
+    )
+    (fp_line (start 1.68 0.95) (end -1.68 0.95) (layer F.CrtYd) (width 0.05))
+    (fp_line (start 1.68 -0.95) (end 1.68 0.95) (layer F.CrtYd) (width 0.05))
+    (fp_line (start -1.68 -0.95) (end 1.68 -0.95) (layer F.CrtYd) (width 0.05))
+    (fp_line (start -1.68 0.95) (end -1.68 -0.95) (layer F.CrtYd) (width 0.05))
+    (fp_line (start -0.258578 0.71) (end 0.258578 0.71) (layer F.SilkS) (width 0.12))
+    (fp_line (start -0.258578 -0.71) (end 0.258578 -0.71) (layer F.SilkS) (width 0.12))
+    (fp_line (start 1 0.6) (end -1 0.6) (layer F.Fab) (width 0.1))
+    (fp_line (start 1 -0.6) (end 1 0.6) (layer F.Fab) (width 0.1))
+    (fp_line (start -1 -0.6) (end 1 -0.6) (layer F.Fab) (width 0.1))
+    (fp_line (start -1 0.6) (end -1 -0.6) (layer F.Fab) (width 0.1))
+    (pad 2 smd roundrect (at 0.9375 0 90) (size 0.975 1.4) (layers F.Cu F.Paste F.Mask) (roundrect_rratio 0.25)
+      (net 3 GND))
+    (pad 1 smd roundrect (at -0.9375 0 90) (size 0.975 1.4) (layers F.Cu F.Paste F.Mask) (roundrect_rratio 0.25)
+      (net 138 SYS_VOUT))
+    (model ${KISYS3DMOD}/Capacitor_SMD.3dshapes/C_0805_2012Metric.wrl
+      (at (xyz 0 0 0))
+      (scale (xyz 1 1 1))
+      (rotate (xyz 0 0 0))
+    )
   )
   (module lichen-badge:LED_SunLED_PLCC4_3.2x2.8mm_Reverse_Mount (layer F.Cu)
@@
       (at (xyz 0 0 0))
       (scale (xyz 1 1 1))
-      (rotate (xyz 0 0 0))
-    )
-  )
-  (module Inductor_SMD:L_0805_2012Metric (layer F.Cu)
-    (at 94.488 119.8118 90)
-    (descr "Inductor SMD 0805 (2012 Metric), square (rectangular) end terminal, IPC_7351 nominal, (Body size source: https://docs.google.com/spreadsheets/d/1BsfQQcO9C6DZCsRaXUlFlo91Tg2WpOkGARC1WS5S8t0/edit?usp=sharing), generated with kicad-footprint-generator")
-    (tags inductor)
-    (attr smd)
-    (fp_text reference C9 (at 2.794 0.0508 90) (layer F.SilkS)
-      (effects (font (size 1 1) (thickness 0.15)))
-    )
-    (fp_text value 47uF (at 0 1.65 90) (layer F.Fab)
-      (effects (font (size 1 1) (thickness 0.15)))
-    )
-    (fp_text user %R (at 0 0 90) (layer F.Fab)
-      (effects (font (size 0.5 0.5) (thickness 0.08)))
-    )
-    (fp_line (start 1.68 0.95) (end -1.68 0.95) (layer F.CrtYd) (width 0.05))
-    (fp_line (start 1.68 -0.95) (end 1.68 0.95) (layer F.CrtYd) (width 0.05))
-    (fp_line (start -1.68 -0.95) (end 1.68 -0.95) (layer F.CrtYd) (width 0.05))
-    (fp_line (start -1.68 0.95) (end -1.68 -0.95) (layer F.CrtYd) (width 0.05))
-    (fp_line (start -0.258578 0.71) (end 0.258578 0.71) (layer F.SilkS) (width 0.12))
-    (fp_line (start -0.258578 -0.71) (end 0.258578 -0.71) (layer F.SilkS) (width 0.12))
-    (fp_line (start 1 0.6) (end -1 0.6) (layer F.Fab) (width 0.1))
-    (fp_line (start 1 -0.6) (end 1 0.6) (layer F.Fab) (width 0.1))
-    (fp_line (start -1 -0.6) (end 1 -0.6) (layer F.Fab) (width 0.1))
-    (fp_line (start -1 0.6) (end -1 -0.6) (layer F.Fab) (width 0.1))
-    (pad 2 smd roundrect (at 0.9375 0 90) (size 0.975 1.4) (layers F.Cu F.Paste F.Mask) (roundrect_rratio 0.25)
-      (net 3 GND))
-    (pad 1 smd roundrect (at -0.9375 0 90) (size 0.975 1.4) (layers F.Cu F.Paste F.Mask) (roundrect_rratio 0.25)
-      (net 138 SYS_VOUT))
-    (model ${KISYS3DMOD}/Inductor_SMD.3dshapes/L_0805_2012Metric.wrl
-      (at (xyz 0 0 0))
-      (scale (xyz 1 1 1))
